File: StepTruck_Esquematico.brd (EAGLE design)
At the start: 70.8 x 43.2 mm, 34 parts, among them U1 ADS1246IPWR, U2 STM32F103C8T6, U3 USB4105-GF-A, U4 C5SMF-RJE-CT0W0BB2, U5 APA2107QWF/D, U6 TS104TAA, U7 XC6206P33MR-G, U8 PTS526, X1 MKDSN1,5/2-5,08

Commit message: Entregable PCB
Parts:
- moved U4 19.0 mm to (65.3, 32.6)
- moved U6 13.6 mm to (38.7, 20.3), turned to 270 degrees
- moved R9 6.72 mm to (41.7, 44.1)
- moved X1 5.08 mm to (65.4, 43.8), turned to 270 degrees
- moved R7 4.69 mm to (39.1, 44.1)
- moved R8 3.59 mm to (36.6, 44.1)
- moved R6 3.41 mm to (44.2, 44.1)
- moved R10 2.54 mm to (31.9, 44.1)
- moved R11 2.54 mm to (28.1, 44.1)
- moved R13 1.80 mm to (50.4, 56.3)
- moved C10 1.27 mm to (35.2, 53.3)
- moved R15 1.09 mm to (44.6, 51.2)
Connections:
- net GND: now also U8.PIN1, U8.PIN2; no longer U8.1, U8.3
- net NRST: now also U8.PIN3, U8.PIN4; no longer U8.2, U8.4
Routing:
- net +3V3: track 13.1 -> 168.7 mm, vias 0 -> 9
- net NRST: track 0.00 -> 69.5 mm, vias 0 -> 6
- net +5V: track 26.0 -> 68.9 mm, vias 2 -> 4
- net PB7: track 0.00 -> 33.7 mm
- net N$17: track 0.00 -> 32.6 mm, vias 0 -> 2
- net N$7: track 0.00 -> 26.8 mm, vias 0 -> 2
- net N$14: track 0.00 -> 25.3 mm
- net SWDIO: track 0.00 -> 22.5 mm, vias 0 -> 2
- net N$2: track 0.00 -> 21.1 mm, vias 0 -> 2
- net N$13: track 0.00 -> 20.9 mm
- net N$4: track 0.00 -> 20.9 mm
- net ADS_START: track 0.00 -> 19.0 mm, vias 0 -> 2
- net ADS_NCS: track 0.00 -> 18.5 mm, vias 0 -> 2
- net N$10: track 0.00 -> 16.4 mm, vias 0 -> 2
- net N$3: track 0.00 -> 15.9 mm, vias 0 -> 2
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Other:
- board text added: "G2 STEPTRACK ELO301 2023"
- board text added: "INPUT"
