File: StepTruck_Esquematico.sch (EAGLE design)
At the start: 34 parts, among them U1 ADS1246IPWR, U2 STM32F103C8T6, U3 USB4105-GF-A, X1 MKDSN1,5/2-5,08

Commit message: Actualizacion Esquematico
Parts:
- removed U$1: APA2107QWF/D, LED_BLANCO:APA2107QWF/D
- removed U$2: C5SMF-RJE-CT0W0BB2, LED_ROJO:C5SMF-RJE-CT0W0BB2
- removed U$3: XC6206P33MR-G, XC6206P332MR-G-TS:XC6206P33MR-G
- removed U$6: TS104TAA, SWD:TS104TAA
- removed U$7: PTS526, PTS526:PTS526
- added U4: C5SMF-RJE-CT0W0BB2, LED_ROJO:C5SMF-RJE-CT0W0BB2
- added U5: APA2107QWF/D, LED_BLANCO:APA2107QWF/D
- added U6: TS104TAA, SWD:TS104TAA
- added U7: XC6206P33MR-G, XC6206P332MR-G-TS:XC6206P33MR-G
- added U8: PTS526, PTS526:PTS526
Connections:
- net +3V3: now also U2PWR.VBAT, U2PWR.VDDA, U2PWR.VDD_1, U2PWR.VDD_2, U2PWR.VDD_3, U5.ANODE, U6.VCC3V3, U7.VOUT; no longer U$1.ANODE, U$3.VOUT, U$6.VCC3V3, U2U2.VBAT, U2U2.VDDA, U2U2.VDD_1, U2U2.VDD_2, U2U2.VDD_3
- net +5V: now also U7.VIN; no longer U$3.VIN
- net ADS_NCS: now also U2MCU.PA4; no longer U2U1.PA4
- net ADS_NDRDY: now also U2MCU.PB0; no longer U2U1.PB0
- net ADS_START: now also U2MCU.PA3; no longer U2U1.PA3
- net GND: now also U2PWR.VSSA, U2PWR.VSS_1, U2PWR.VSS_2, U2PWR.VSS_3, U6.GND, U7.VSS, U8.PIN1, U8.PIN3; no longer U$3.VSS, U$6.GND, U$7.PIN1, U$7.PIN3, U2U2.VSSA, U2U2.VSS_1, U2U2.VSS_2, U2U2.VSS_3
- net MISO: now also U2MCU.PA6; no longer U2U1.PA6
- net MOSI: now also U2MCU.PA7; no longer U2U1.PA7
- net N$5: now also U5.CATHODE; no longer U$1.CATHODE
- net N$6: now also U4.OUT-; no longer U$2.OUT-
- net NRST: now also U2MCU.NRST, U8.PIN2, U8.PIN4; no longer U$7.PIN2, U$7.PIN4, U2U1.NRST
- net PA11: now also U2MCU.PA11; no longer U2U1.PA11
- net PA12: now also U2MCU.PA12; no longer U2U1.PA12
- net PB7: now also U2MCU.PB7, U4.+IN; no longer U$2.+IN, U2U1.PB7
- net SCLK: now also U2MCU.PA5; no longer U2U1.PA5
- net SWDCLK: now also U2MCU.PA14, U6.SWDCLK; no longer U$6.SWDCLK, U2U1.PA14
- net SWDIO: now also U2MCU.PA13, U6.SWDIO; no longer U$6.SWDIO, U2U1.PA13
Other:
- note added: "Vmax:"
- note added: "Vmin:"

Commit message: Entregable PCB
Connections:
- net GND: now also U8.PIN2; no longer U8.PIN3
- net NRST: now also U8.PIN3; no longer U8.PIN2
Changed lines of the file:
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@@
 <junction x="-91.44" y="-175.26"/>
 <pinref part="U8" gate="BOTON" pin="PIN1"/>
-<pinref part="U8" gate="BOTON" pin="PIN3"/>
+<pinref part="U8" gate="BOTON" pin="PIN2"/>
 </segment>
 </net>
@@
 <wire x1="-91.44" y1="-144.78" x2="-86.36" y2="-144.78" width="0.1524" layer="91"/>
 <junction x="-67.31" y="-144.78"/>
-<pinref part="U8" gate="BOTON" pin="PIN2"/>
+<pinref part="U8" gate="BOTON" pin="PIN3"/>
 <pinref part="U8" gate="BOTON" pin="PIN4"/>
 <wire x1="-86.36" y1="-144.78" x2="-67.31" y2="-144.78" width="0.1524" layer="91"/>
